Commit message: rotate camera

File: hector_quadrotor/hector_quadrotor_description/urdf/quadrotor_hokuyo_utm30lx.urdf.xacro (robot description, xacro)
@@ -13,6 +13,6 @@
     <!-- Forward facing camera -->
     <xacro:include filename="$(find hector_sensors_description)/urdf/generic_camera.urdf.xacro" />
-    <xacro:generic_camera name="front_cam" parent="base_link" ros_topic="camera/image" cam_info_topic="camera/camera_info" update_rate="30" res_x="640" res_y="480" image_format="R8G8B8" hfov="90">
-      <origin xyz="0.05 -0.0 -0.25" rpy="0 0 0"/>
+    <xacro:generic_camera name="front_cam" parent="base_link" ros_topic="camera/image" cam_info_topic="camera/camera_info" update_rate="30" res_x="1280" res_y="720" image_format="R8G8B8" hfov="90">
+      <origin xyz="0.0 0.0 -0.1" rpy="0 1.5708 0"/>
     </xacro:generic_camera>
 </robot>
